File: sensorHub.sch (EAGLE design)
At the start: 0 parts

Commit message: Adds the feather m0 to schematic
Parts:
- added JP1: (no value), pinhead:PINHD-2X16
- added JP2: (no value), pinhead:PINHD-2X11
- added MS1: FEATHERWING, adafruit:FEATHERWING
